Commit message: feat(bringup): add ROS 2 Humble bootstrap scripts, bring-up package, and docs; fix EKF YAML and minimal URDF; add diagnostics
- scripts/bootstrap_ros2_humble.sh (idempotent ROS 2 install for Ubuntu 22.04)
- scripts/check_stack.sh (quick health check)
- docs/bringup/os_ros.md: concrete install steps
- bringup/alpha_viam_bringup: ament_python package with base_bringup.launch.py
- configs/ekf.yaml: proper ros__parameters structure
- urdf/rover.urdf.xacro: minimal base_link to start RSP
- launch composes robot_state_publisher, EKF, diagnostic_aggregator, foxglove_bridge
- add .gitignore to exclude build/install/log

File: urdf/rover.urdf.xacro (robot description, xacro)
@@ -1,5 +1,26 @@
 <?xml version="1.0"?>
 <robot xmlns:xacro="http://www.ros.org/wiki/xacro" name="alpha_viam_rover">
-  <!-- Placeholder URDF/Xacro. Add links, joints, and ros2_control tags. -->
-  <xacro:macro name="base" params="prefix:=''"></xacro:macro>
+  <!-- Minimal URDF: single base_link with simple geometry -->
+  <link name="base_link">
+    <inertial>
+      <origin xyz="0 0 0" rpy="0 0 0"/>
+      <mass value="2.0"/>
+      <inertia ixx="0.02" ixy="0.0" ixz="0.0" iyy="0.02" iyz="0.0" izz="0.04"/>
+    </inertial>
+    <visual>
+      <origin xyz="0 0 0.05" rpy="0 0 0"/>
+      <geometry>
+        <box size="0.25 0.18 0.10"/>
+      </geometry>
+      <material name="grey">
+        <color rgba="0.5 0.5 0.5 1.0"/>
+      </material>
+    </visual>
+    <collision>
+      <origin xyz="0 0 0.05" rpy="0 0 0"/>
+      <geometry>
+        <box size="0.25 0.18 0.10"/>
+      </geometry>
+    </collision>
+  </link>
 </robot>

Commit message: feat(urdf): add base/wheels/sensor links and joints; add TF contract doc (resolve base_link geometry)

File: urdf/rover.urdf.xacro (robot description, xacro)
@@ -1,5 +1,9 @@
 <?xml version="1.0"?>
 <robot xmlns:xacro="http://www.ros.org/wiki/xacro" name="alpha_viam_rover">
-  <!-- Minimal URDF: single base_link with simple geometry -->
+  <!-- Minimal URDF/Xacro for TF and diff-drive semantics. Dimensions are placeholders. -->
+  <!-- Parameters -->
+  <xacro:property name="wheel_separation" value="0.30"/>
+  <xacro:property name="wheel_radius" value="0.06"/>
+  <!-- Base with simple geometry/inertial -->
   <link name="base_link">
     <inertial>
@@ -24,3 +28,32 @@
     </collision>
   </link>
+  <!-- Wheels -->
+  <link name="left_wheel_link"/>
+  <link name="right_wheel_link"/>
+  <joint name="left_wheel_joint" type="continuous">
+    <parent link="base_link"/>
+    <child link="left_wheel_link"/>
+    <origin xyz="0 ${wheel_separation/2.0} 0" rpy="0 0 0"/>
+    <axis xyz="0 1 0"/>
+  </joint>
+  <joint name="right_wheel_joint" type="continuous">
+    <parent link="base_link"/>
+    <child link="right_wheel_link"/>
+    <origin xyz="0 ${-wheel_separation/2.0} 0" rpy="0 0 0"/>
+    <axis xyz="0 1 0"/>
+  </joint>
+  <!-- Sensors -->
+  <link name="imu_link"/>
+  <joint name="imu_joint" type="fixed">
+    <parent link="base_link"/>
+    <child link="imu_link"/>
+    <origin xyz="0 0 0.05" rpy="0 0 0"/>
+  </joint>
+  <link name="lidar_link"/>
+  <joint name="lidar_joint" type="fixed">
+    <parent link="base_link"/>
+    <child link="lidar_link"/>
+    <origin xyz="0.10 0 0.08" rpy="0 0 0"/>
+  </joint>
+  <!-- Placeholder for ros2_control tags (controllers/hardware will be added later). -->
 </robot>

Commit message: feat(urdf): add ros2_control system/joint interfaces and placeholder transmissions to match diff_drive joints

File: urdf/rover.urdf.xacro (robot description, xacro)
@@ -56,4 +56,41 @@
     <origin xyz="0.10 0 0.08" rpy="0 0 0"/>
   </joint>
-  <!-- Placeholder for ros2_control tags (controllers/hardware will be added later). -->
+  <!-- ros2_control: system + joint interfaces (placeholders for real hardware) -->
+  <ros2_control name="RoverSystem" type="system">
+    <hardware>
+      <!-- Placeholder hardware plugin; replace with real hardware when available -->
+      <plugin>mock_components/GenericSystem</plugin>
+    </hardware>
+    <joint name="left_wheel_joint">
+      <command_interface name="velocity"/>
+      <state_interface name="position"/>
+      <state_interface name="velocity"/>
+    </joint>
+    <joint name="right_wheel_joint">
+      <command_interface name="velocity"/>
+      <state_interface name="position"/>
+      <state_interface name="velocity"/>
+    </joint>
+  </ros2_control>
+  <!-- Optional transmissions for tooling compatibility (placeholder) -->
+  <transmission name="left_wheel_transmission">
+    <type>transmission_interface/SimpleTransmission</type>
+    <joint name="left_wheel_joint">
+      <hardwareInterface>hardware_interface/VelocityJointInterface</hardwareInterface>
+    </joint>
+    <actuator name="left_motor">
+      <hardwareInterface>hardware_interface/VelocityJointInterface</hardwareInterface>
+      <mechanicalReduction>1.0</mechanicalReduction>
+    </actuator>
+  </transmission>
+  <transmission name="right_wheel_transmission">
+    <type>transmission_interface/SimpleTransmission</type>
+    <joint name="right_wheel_joint">
+      <hardwareInterface>hardware_interface/VelocityJointInterface</hardwareInterface>
+    </joint>
+    <actuator name="right_motor">
+      <hardwareInterface>hardware_interface/VelocityJointInterface</hardwareInterface>
+      <mechanicalReduction>1.0</mechanicalReduction>
+    </actuator>
+  </transmission>
 </robot>
